Commit message: Replace "base" with "GUI_base", replace "map" with "GUI_map"

File: src/visualization/opengl_test/geometry_description/urdf/ICLU_B1.xacro (robot description, xacro)
@@ -2,10 +2,10 @@
 <robot name="ADV" xmlns:xacro="http://www.ros.org/wiki/xacro">
     <!-- base frame (lidar) -->
-    <link name="base">
+    <link name="GUI_base">
     </link>
     <!-- base frame (lidar frame) to the footprint (ground level) -->
     <joint name="base_joint" type="fixed">
         <origin xyz="0 0 -3.0" rpy="0 0 0" />
-        <parent link="base"/>
+        <parent link="GUI_base"/>
         <child link="GUI_base_footprint" />
     </joint>

File: src/visualization/opengl_test/geometry_description/urdf/world_flower_expo.xacro (robot description, xacro)
@@ -2,10 +2,10 @@
 <robot name="world" xmlns:xacro="http://www.ros.org/wiki/xacro">
     <!-- map frame -->
-    <link name="map">
+    <link name="GUI_map">
     </link>
     <!-- GUI_NLOS frame -->
     <joint name="NLOS_joint" type="fixed">
         <origin xyz="0 0 -3.0" rpy="0 0 0" />
-        <parent link="map"/>
+        <parent link="GUI_map"/>
         <child link="GUI_NLOS" />
     </joint>
