Commit message: update planning module and vehicle module

File: src/vehicle/vehicle_description/vehicle_body_description/b_bus_description/urdf/b_bus.xacro (robot description, xacro)
@@ -6,5 +6,5 @@
   <link name="base_link">
     <visual>
-      <origin xyz="-1.7 0 1.5" rpy="${pi/2.0} 0 ${pi}"/>
+      <origin xyz="-5.85 0 0" rpy="${pi/2.0} 0 ${pi}"/>
       <geometry>
         <mesh filename="package://b_bus_description/mesh/b_bus.dae" scale="1 1 1"/>
