Commit message: update vehicle description and fix map(traffic light)

File: src/launcher/vehicle_launch/urdf/vehicle.xacro (robot description, xacro)
@@ -3,9 +3,9 @@
   xmlns:xacro="http://ros.org/wiki/xacro">
   <xacro:include filename="$(find b_bus_description)/urdf/b_bus.xacro"/>
-  <xacro:include filename="$(find vehicle_launch)/urdf/sensor_kit.xacro"/>
-  <xacro:property name="calibration" value="${load_yaml('$(find vehicle_launch)/config/sensors_calibration.yaml')}"/>
+  <!--xacro:include filename="$(find vehicle_launch)/urdf/sensor_kit.xacro"/-->
+  <!--xacro:property name="calibration" value="${load_yaml('$(find vehicle_launch)/config/sensors_calibration.yaml')}"/-->
   <!-- sensor_kit -->
-  <xacro:sensor_kit_macro parent="base_link" x="${calibration['base_link2sensor_kit_base_link']['x']}" y="${calibration['base_link2sensor_kit_base_link']['y']}" z="${calibration['base_link2sensor_kit_base_link']['z']}" roll="${calibration['base_link2sensor_kit_base_link']['roll']}" pitch="${calibration['base_link2sensor_kit_base_link']['pitch']}" yaw="${calibration['base_link2sensor_kit_base_link']['yaw']}" />
+  <!--xacro:sensor_kit_macro parent="base_link" x="${calibration['base_link2sensor_kit_base_link']['x']}" y="${calibration['base_link2sensor_kit_base_link']['y']}" z="${calibration['base_link2sensor_kit_base_link']['z']}" roll="${calibration['base_link2sensor_kit_base_link']['roll']}" pitch="${calibration['base_link2sensor_kit_base_link']['pitch']}" yaw="${calibration['base_link2sensor_kit_base_link']['yaw']}" /-->
   <!-- gnss -->
-  <xacro:imu_macro suffix="gnss" parent="base_link" namespace="" x="${calibration['base_link2gnss']['x']}" y="${calibration['base_link2gnss']['y']}" z="${calibration['base_link2gnss']['z']}" roll="${calibration['base_link2gnss']['roll']}" pitch="${calibration['base_link2gnss']['pitch']}" yaw="${calibration['base_link2gnss']['yaw']}" fps="100" />
+  <!--xacro:imu_macro suffix="gnss" parent="base_link" namespace="" x="${calibration['base_link2gnss']['x']}" y="${calibration['base_link2gnss']['y']}" z="${calibration['base_link2gnss']['z']}" roll="${calibration['base_link2gnss']['roll']}" pitch="${calibration['base_link2gnss']['pitch']}" yaw="${calibration['base_link2gnss']['yaw']}" fps="100" /-->
 </robot>
